Commit message: debugged and fixed issue with continuous thigh joints causing position error. Switch out urdfs to one with revolute joints

File: resources/robots/aliengo/urdf/aliengo.urdf (robot description, URDF)
Before this commit: robot aliengo_description, 17 links, 16 joints
Links:
- added link base; visual box size=0.001 0.001 0.001
- added link imu_link, mass 0.001; collision box size=.001 .001 .001; visual box size=0.001 0.001 0.001
- link FL_calf: geometry collision box size=0.25 0.0208 0.016; visual mesh filename=../meshes/calf.dae scale=1 1 1
- link FL_hip: geometry collision cylinder length=0.0418 radius=0.046; visual mesh filename=../meshes/hip.dae scale=1 1 1
- link FL_thigh: geometry collision box size=0.25 0.0374 0.043; visual mesh filename=../meshes/thigh.dae scale=1 1 1
- link FR_calf: geometry collision box size=0.25 0.0208 0.016; visual mesh filename=../meshes/calf.dae scale=1 1 1
- link FR_hip: geometry collision cylinder length=0.0418 radius=0.046; visual mesh filename=../meshes/hip.dae scale=1 1 1
- link FR_thigh: geometry collision box size=0.25 0.0374 0.043; visual mesh filename=../meshes/thigh_mirror.dae scale=1 1 1
- link RL_calf: geometry collision box size=0.25 0.0208 0.016; visual mesh filename=../meshes/calf.dae scale=1 1 1
- link RL_hip: geometry collision cylinder length=0.0418 radius=0.046; visual mesh filename=../meshes/hip.dae scale=1 1 1
- link RL_thigh: geometry collision box size=0.25 0.0374 0.043; visual mesh filename=../meshes/thigh.dae scale=1 1 1
- link RR_calf: geometry collision box size=0.25 0.0208 0.016; visual mesh filename=../meshes/calf.dae scale=1 1 1
- link RR_hip: geometry collision cylinder length=0.0418 radius=0.046; visual mesh filename=../meshes/hip.dae scale=1 1 1
- link RR_thigh: geometry collision box size=0.25 0.0374 0.043; visual mesh filename=../meshes/thigh_mirror.dae scale=1 1 1
- link trunk: geometry collision box size=0.647 0.15 0.112; visual mesh filename=../meshes/trunk.dae scale=1 1 1
Joints:
- added joint floating_base: type fixed, parent base, child trunk, origin xyz=0 0 0 rpy=0 0 0
- added joint imu_joint: type fixed, parent trunk, child imu_link, origin xyz=0 0 0 rpy=0 0 0
- joint FL_calf_joint: limit lower=-2.77507351067 upper=-0.645771823238 effort=44.4 velocity=40 -> lower=-2.77507351067 upper=-0.645771823238 effort=55 velocity=16
- joint FL_hip_joint: limit lower=-1.2217304764 upper=1.2217304764 effort=44.4 velocity=40 -> lower=-1.2217304764 upper=1.2217304764 effort=44 velocity=20
- joint FL_thigh_joint: limit effort=44.4 velocity=40 -> lower=-1.0471975512 upper=4.18879020479 effort=44 velocity=20; type continuous -> revolute
- joint FR_calf_joint: limit lower=-2.77507351067 upper=-0.645771823238 effort=44.4 velocity=40 -> lower=-2.77507351067 upper=-0.645771823238 effort=55 velocity=16
- joint FR_hip_joint: limit lower=-1.2217304764 upper=1.2217304764 effort=44.4 velocity=40 -> lower=-1.2217304764 upper=1.2217304764 effort=44 velocity=20
- joint FR_thigh_joint: limit effort=44.4 velocity=40 -> lower=-1.0471975512 upper=4.18879020479 effort=44 velocity=20; type continuous -> revolute
- joint RL_calf_joint: limit lower=-2.77507351067 upper=-0.645771823238 effort=44.4 velocity=40 -> lower=-2.77507351067 upper=-0.645771823238 effort=55 velocity=16
- joint RL_hip_joint: limit lower=-1.2217304764 upper=1.2217304764 effort=44.4 velocity=40 -> lower=-1.2217304764 upper=1.2217304764 effort=44 velocity=20
- joint RL_thigh_joint: limit effort=44.4 velocity=40 -> lower=-1.0471975512 upper=4.18879020479 effort=44 velocity=20; type continuous -> revolute
- joint RR_calf_joint: limit lower=-2.77507351067 upper=-0.645771823238 effort=44.4 velocity=40 -> lower=-2.77507351067 upper=-0.645771823238 effort=55 velocity=16
- joint RR_hip_joint: limit lower=-1.2217304764 upper=1.2217304764 effort=44.4 velocity=40 -> lower=-1.2217304764 upper=1.2217304764 effort=44 velocity=20
- joint RR_thigh_joint: limit effort=44.4 velocity=40 -> lower=-1.0471975512 upper=4.18879020479 effort=44 velocity=20; type continuous -> revolute
